File: pcb/Angel Wings v.2.1/Angel Wings FINAL.kicad_pcb (KiCad board)
At the start: 2 copper layers, 153.9 x 93.7 mm, 82 parts, among them J1 MJ-4PP-9-kbd, SW1 SW_PUSH-kbd, SW10 SW_PUSH-kbd, SW11 SW_PUSH-kbd, SW12 SW_PUSH-kbd, SW13 SW_PUSH-kbd, SW14 SW_PUSH-kbd, SW15 SW_PUSH-kbd, SW16 SW_PUSH-kbd, SW17 SW_PUSH-kbd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

Commit message: fix AWF v.2.1
Routing:
- net Col 0: track 263.4 -> 253.5 mm, vias 2 -> 3
- net VCC: track 756.6 -> 753.6 mm
- net Row 0: track 257.7 -> 256.6 mm
- net Row 1: track 241.8 -> 241.6 mm, vias 2 -> 4
- net GND: vias 29 -> 59
Other:
- outline, holes or cut-outs redrawn
